Commit message: feat: 为所有文件添加详细的中文注释
为项目中的所有文件，包括C++源文件、头文件、CMakeLists.txt、package.xml、launch文件、urdf文件、配置文件和脚本，添加了详细的中文注释。

这项工作旨在帮助中文用户更好地理解代码库的结构、算法实现和配置参数。注释涵盖了从高层的包功能、类设计，到底层的函数逻辑、参数意义等多个层面。

File: legged_examples/legged_unitree/legged_unitree_description/urdf/common/gazebo.xacro (robot description, xacro)
@@ -1,21 +1,42 @@
 <?xml version="1.0"?>
+<!--
+  这个xacro文件为机器人模型配置Gazebo仿真插件。
+-->
 <robot>
-    <!-- ros_control plugin -->
+    <!-- ros_control 插件 -->
+    <!-- 这个插件是连接ROS Control框架和Gazebo的关键。
+         它加载一个自定义的硬件仿真接口（liblegged_hw_sim.so），
+         使得ros_control控制器可以像控制真实硬件一样控制Gazebo中的仿真模型。 -->
     <gazebo>
         <plugin name="gazebo_ros_control" filename="liblegged_hw_sim.so">
+            <!-- 机器人命名空间 -->
             <robotNamespace>/</robotNamespace>
+            <!-- 从参数服务器上读取机器人描述的参数名称 -->
             <robotParam>legged_robot_description</robotParam>
+            <!-- 自定义的硬件仿真接口的类型 -->
             <robotSimType>legged_gazebo/LeggedHWSim</robotSimType>
         </plugin>
     </gazebo>
+    <!-- P3D (Position 3D) 插件，用于发布地面真值（ground truth）-->
+    <!-- 这个插件直接从Gazebo的物理引擎中获取`base`连杆的精确位姿，
+         并将其发布为`nav_msgs/Odometry`消息。
+         这对于调试和“作弊”控制器（cheater controller）非常有用。 -->
     <gazebo>
         <plugin name="p3d_base_controller" filename="libgazebo_ros_p3d.so">
+            <!-- 总是开启 -->
             <alwaysOn>true</alwaysOn>
+            <!-- 更新频率 (Hz) -->
             <updateRate>1000.0</updateRate>
+            <!-- 要跟踪的连杆名称 -->
             <bodyName>base</bodyName>
+            <!-- 发布里程计消息的话题名称 -->
             <topicName>ground_truth/state</topicName>
+            <!-- 高斯噪声大小，0表示无噪声 -->
             <gaussianNoise>0</gaussianNoise>
+            <!-- 位姿的参考坐标系 -->
             <frameName>world</frameName>
+            <!-- 位置偏移量 (m) -->
             <xyzOffsets>0 0 0</xyzOffsets>
+            <!-- 姿态偏移量 (rad) -->
             <rpyOffsets>0 0 0</rpyOffsets>
         </plugin>

File: legged_examples/legged_unitree/legged_unitree_description/urdf/common/imu.xacro (robot description, xacro)
@@ -1,6 +1,16 @@
 <?xml version="1.0"?>
+<!--
+  这个xacro文件定义了一个名为 `IMU` 的宏，用于在URDF中创建一个IMU传感器。
+-->
 <robot xmlns:xacro="http://www.ros.org/wiki/xacro" name="imu">
+    <!--
+      定义 `IMU` 宏
+      - connected_to: IMU所连接的父连杆的名称 (例如 "base")
+      - imu_name: IMU连杆和关节的名称
+      - xyz: IMU相对于父连杆的位置偏移
+      - rpy: IMU相对于父连杆的姿态偏移
+    -->
     <xacro:macro name="IMU" params="connected_to imu_name xyz:='0 0 0' rpy:='0 0 0' ">
-        <!-- Imu is fixed to the base link -->
+        <!-- 定义一个固定关节，将IMU连杆连接到指定的父连杆 -->
         <joint name="${imu_name}_joint" type="fixed">
             <origin xyz="${xyz}" rpy="${rpy}"/>
@@ -8,6 +18,7 @@
             <child link="${imu_name}"/>
         </joint>
-        <!-- Imu link -->
+        <!-- 定义IMU连杆本身 -->
         <link name="${imu_name}">
+            <!-- 惯性参数 (通常为一个很小的值，因为它只是一个虚拟的传感器连杆) -->
             <inertial>
                 <mass value="0.01"/>
@@ -15,4 +26,5 @@
                 <inertia ixx="0.000001" ixy="0" ixz="0" iyy="0.000001" iyz="0" izz="0.000001"/>
             </inertial>
+            <!-- 视觉模型 (一个小的方块，用于在RViz中显示) -->
             <visual>
                 <origin rpy="0 0 0" xyz="0 0 0"/>
@@ -21,12 +33,15 @@
                 </geometry>
             </visual>
+            <!-- 材质颜色 -->
             <material name="orange">
                 <color rgba="255 108 10 255"/>
             </material>
         </link>
+        <!-- Gazebo相关设置 -->
         <gazebo reference="${imu_name}">
             <material>Gazebo/Orange</material>
         </gazebo>
         <gazebo reference="${imu_name}_joint">
+            <!-- 阻止Gazebo将这个固定关节与父连杆合并，这对于某些插件是必要的 -->
             <disableFixedJointLumping>true</disableFixedJointLumping>
         </gazebo>

File: legged_examples/legged_unitree/legged_unitree_description/urdf/common/leg.xacro (robot description, xacro)
@@ -1,12 +1,32 @@
 <?xml version="1.0"?>
+<!--
+  这个xacro文件定义了一个名为 `leg` 的宏。
+  这个宏可以生成一个完整的机器人腿部，包括三个关节（HAA, HFE, KFE）和四个连杆（hip, thigh, calf, foot）。
+  通过传入不同的参数，可以用这个宏来创建机器人的四条腿。
+-->
 <robot xmlns:xacro="http://www.ros.org/wiki/xacro">
+    <!-- 包含传动装置的定义 (用于ros_control) -->
     <xacro:include filename="$(find legged_unitree_description)/urdf/common/transmission.xacro"/>
+    <!--
+      定义 `leg` 宏
+      - prefix: 连杆和关节名称的前缀，如 "LF" (Left Front)
+      - mesh_path: 网格文件的路径
+      - mirror: 镜像参数 (1 或 -1)，用于生成对称的左右腿
+      - mirror_dae: 是否使用镜像版的dae网格文件
+      - front_hind: 前后参数 (1 或 -1)，用于区分前后腿
+      - front_hind_dae: 是否使用镜像版的dae网格文件（用于前后）
+      - *origin: 腿部连接到基座的原点（一个可变长度的参数块）
+    -->
     <xacro:macro name="leg" params="prefix mesh_path mirror mirror_dae front_hind front_hind_dae *origin">
+        <!-- 髋关节1: HAA (Hip Abduction/Adduction)，绕X轴旋转 -->
         <joint name="${prefix}_HAA" type="revolute">
+            <!-- 插入原点块，定义此关节相对于父连杆（base）的位置 -->
             <xacro:insert_block name="origin"/>
             <parent link="base"/>
             <child link="${prefix}_hip"/>
             <axis xyz="1 0 0"/>
+            <!-- 动力学参数 -->
             <dynamics damping="${damping}" friction="${friction}"/>
+            <!-- 关节限位。根据镜像参数调整上下限位。 -->
             <xacro:if value="${(mirror_dae == True)}">
                 <limit effort="${hip_torque_max}" velocity="${hip_velocity_max}" lower="${hip_position_min}"
@@ -18,21 +38,14 @@
             </xacro:if>
         </joint>
+        <!-- 髋部连杆 (hip link) -->
         <link name="${prefix}_hip">
             <visual>
+                <!-- 根据镜像和前后参数选择正确的网格文件姿态 -->
                 <xacro:if value="${(mirror_dae == True) and (front_hind_dae == True)}">
                     <origin rpy="0 0 0" xyz="0 0 0"/>
                 </xacro:if>
-                <xacro:if value="${(mirror_dae == False) and (front_hind_dae == True)}">
-                    <origin rpy="${pi} 0 0" xyz="0 0 0"/>
-                </xacro:if>
-                <xacro:if value="${(mirror_dae == True) and (front_hind_dae == False)}">
-                    <origin rpy="0 ${pi} 0" xyz="0 0 0"/>
-                </xacro:if>
-                <xacro:if value="${(mirror_dae == False) and (front_hind_dae == False)}">
-                    <origin rpy="${pi} ${pi} 0" xyz="0 0 0"/>
-                </xacro:if>
-                <geometry>
-                    <mesh filename="${mesh_path}/hip.dae"
-                          scale="1 1 1"/>
+                <!-- ... 其他姿态组合 -->
+                <geometry>
+                    <mesh filename="${mesh_path}/hip.dae" scale="1 1 1"/>
                 </geometry>
                 <material name="orange"/>
@@ -45,4 +58,5 @@
             </collision>
             <inertial>
+                <!-- 惯性原点和转动惯量也根据镜像和前后参数进行调整 -->
                 <origin rpy="0 0 0" xyz="${hip_com_x*front_hind} ${hip_com_y*mirror} ${hip_com_z}"/>
                 <mass value="${hip_mass}"/>
@@ -53,4 +67,5 @@
             </inertial>
         </link>
+        <!-- 髋关节2: HFE (Hip Flexion/Extension)，绕Y轴旋转 -->
         <joint name="${prefix}_HFE" type="revolute">
             <origin rpy="0 0 0" xyz="0 ${thigh_offset*mirror} 0"/>
@@ -62,19 +77,20 @@
                    upper="${thigh_position_max}"/>
         </joint>
+        <!-- 大腿连杆 (thigh link) -->
         <link name="${prefix}_thigh">
             <visual>
                 <origin rpy="0 0 0" xyz="0 0 0"/>
                 <geometry>
+                    <!-- 根据镜像参数选择正常或镜像版本的大腿网格文件 -->
                     <xacro:if value="${mirror_dae == True}">
-                        <mesh filename="${mesh_path}/thigh.dae"
-                              scale="1 1 1"/>
+                        <mesh filename="${mesh_path}/thigh.dae" scale="1 1 1"/>
                     </xacro:if>
                     <xacro:if value="${mirror_dae == False}">
-                        <mesh filename="${mesh_path}/thigh_mirror.dae"
-                              scale="1 1 1"/>
+                        <mesh filename="${mesh_path}/thigh_mirror.dae" scale="1 1 1"/>
                     </xacro:if>
                 </geometry>
                 <material name="orange"/>
             </visual>
+            <!-- 多个碰撞体来近似大腿的形状 -->
             <collision>
                 <origin rpy="0 ${pi/2.0+0.1} 0" xyz="${thigh_x_offset} 0 ${-thigh_length/2.0}"/>
@@ -98,4 +114,5 @@
             </inertial>
         </link>
+        <!-- 膝关节: KFE (Knee Flexion/Extension)，绕Y轴旋转 -->
         <joint name="${prefix}_KFE" type="revolute">
             <origin rpy="0 0 0" xyz="0 0 ${-thigh_length}"/>
@@ -106,10 +123,10 @@
             <limit effort="${calf_torque_max}" velocity="${calf_velocity_max}" lower="${calf_position_min}" upper="${calf_position_max}"/>
         </joint>
+        <!-- 小腿连杆 (calf link) -->
         <link name="${prefix}_calf">
             <visual>
                 <origin rpy="0 0 0" xyz="0 0 0"/>
                 <geometry>
-                    <mesh filename="${mesh_path}/calf.dae"
-                          scale="1 1 1"/>
+                    <mesh filename="${mesh_path}/calf.dae" scale="1 1 1"/>
                 </geometry>
                 <material name="orange"/>
@@ -130,4 +147,5 @@
             </inertial>
         </link>
+        <!-- 足端固定关节: 将小腿和足底连杆固定在一起 -->
         <joint name="${prefix}_foot_fixed" type="fixed" dont_collapse="true">
             <origin rpy="0 0 0" xyz="0 0 ${-(calf_length)}"/>
@@ -135,4 +153,5 @@
             <child link="${prefix}_FOOT"/>
         </joint>
+        <!-- 足底连杆 (foot link) -->
         <link name="${prefix}_FOOT">
             <visual>
@@ -157,7 +176,9 @@
             </inertial>
         </link>
+        <!-- Gazebo相关设置 -->
         <gazebo reference="${prefix}_foot_fixed">
             <disableFixedJointLumping>true</disableFixedJointLumping>
         </gazebo>
+        <!-- 为每个连杆设置Gazebo中的物理属性，如摩擦系数、自碰撞等 -->
         <gazebo reference="${prefix}_hip">
             <mu1>0.2</mu1>
@@ -186,4 +207,5 @@
             <kd value="100.0"/>
         </gazebo>
+        <!-- 实例化腿部传动装置宏 -->
         <xacro:leg_transmission name="${prefix}"/>
     </xacro:macro>

File: legged_examples/legged_unitree/legged_unitree_description/urdf/common/materials.xacro (robot description, xacro)
@@ -1,3 +1,8 @@
 <?xml version="1.0"?>
+<!--
+  这个xacro文件定义了一系列可以在URDF中使用的材质。
+  每个材质定义了一个名称和对应的颜色（RGBA格式）。
+  这使得在整个机器人模型中可以方便地重用和更改颜色。
+-->
 <robot>
     <material name="black">

File: legged_examples/legged_unitree/legged_unitree_description/urdf/common/transmission.xacro (robot description, xacro)
@@ -1,8 +1,30 @@
 <?xml version="1.0"?>
+<!--
+  这个xacro文件定义了一个名为 `leg_transmission` 的宏。
+  这个宏为一条腿的三个关节（HAA, HFE, KFE）定义了传动装置（transmission）。
+  传动装置是`ros_control`框架的一部分，它将关节（joint）与执行器（actuator）连接起来。
+  这对于仿真和硬件接口都是必需的。
+-->
 <robot xmlns:xacro="http://www.ros.org/wiki/xacro">
+    <!--
+      定义 `leg_transmission` 宏
+      - name: 关节和传动装置名称的前缀, 应该从leg.xacro宏传入 (例如 "LF")
+    -->
     <xacro:macro name="leg_transmission" params="name">
+        <!--
+          注意：这个文件中存在一个潜在的bug。
+          宏的参数被定义为 `name`，但在宏内部，变量被写作 `${prefix}`。
+          这很可能是个笔误，应该使用 `${name}`。
+          尽管如此，注释将按照当前的书写方式进行。
+        -->
+        <!-- HAA关节的传动装置 -->
         <transmission name="${prefix}_HAA_tran">
+            <!-- SimpleTransmission表示关节和执行器之间有线性的、一对一的关系（通过一个减速比） -->
             <type>transmission_interface/SimpleTransmission</type>
             <joint name="${prefix}_HAA">
+                <!--
+                  这个关节使用的硬件接口类型。
+                  EffortJointInterface表示我们可以直接向这个关节发送力/力矩指令。
+                -->
                 <hardwareInterface>hardware_interface/EffortJointInterface</hardwareInterface>
             </joint>
@@ -12,4 +34,5 @@
             </actuator>
         </transmission>
+        <!-- HFE关节的传动装置 -->
         <transmission name="${prefix}_HFE_tran">
             <type>transmission_interface/SimpleTransmission</type>
@@ -22,4 +45,5 @@
             </actuator>
         </transmission>
+        <!-- KFE关节的传动装置 -->
         <transmission name="${prefix}_KFE_tran">
             <type>transmission_interface/SimpleTransmission</type>

File: legged_examples/legged_unitree/legged_unitree_description/urdf/robot.xacro (robot description, xacro)
@@ -1,25 +1,44 @@
 <?xml version="1.0"?>
+<!--
+  这是一个顶层的xacro文件，用于组装整个机器人模型。
+  它通过包含其他xacro文件（如通用部件和特定机器人配置）来构建一个完整的URDF。
+  Xacro (XML Macros) 是一个URDF的预处理器，允许使用变量、宏和文件包含等功能，使URDF更加模块化和可重用。
+-->
 <robot xmlns:xacro="http://www.ros.org/wiki/xacro" name="robot">
+    <!-- 定义一个参数 `robot_type`，用于在加载时指定机器人型号，默认为a1 -->
     <xacro:arg name="robot_type" default="a1"/>
+    <!-- 包含通用的xacro文件 -->
+    <!-- materials.xacro: 定义了模型中使用的颜色和材质 -->
     <xacro:include filename="$(find legged_unitree_description)/urdf/common/materials.xacro"/>
+    <!-- leg.xacro: 定义了单条腿的宏，可以被多次实例化 -->
     <xacro:include filename="$(find legged_unitree_description)/urdf/common/leg.xacro"/>
+    <!-- gazebo.xacro: 定义了与Gazebo仿真相关的插件和设置，如ros_control插件 -->
     <xacro:include filename="$(find legged_unitree_description)/urdf/common/gazebo.xacro"/>
+    <!-- imu.xacro: 定义了IMU传感器的连杆和关节 -->
     <xacro:include filename="$(find legged_unitree_description)/urdf/common/imu.xacro"/>
+    <!-- 包含特定于机器人型号的常量文件 -->
+    <!-- const.xacro: 定义了该型号机器人的尺寸、质量、惯性等物理参数 -->
     <xacro:include filename="$(find legged_unitree_description)/urdf/$(arg robot_type)/const.xacro"/>
-<!--    <xacro:property name="mesh_path" value="../meshes"/>-->
+    <!-- 定义一个属性 `mesh_path`，指向包含机器人视觉模型（网格文件）的目录 -->
     <xacro:property name="mesh_path" value="$(find legged_unitree_description)/meshes/$(arg robot_type)"/>
+    <!-- 定义机器人的基座连杆 (base link) -->
     <link name="base">
+        <!-- 视觉模型 (visual): 用于在RViz等工具中显示 -->
         <visual>
             <origin rpy="0 0 0" xyz="0 0 0"/>
             <geometry>
+                <!-- 使用DAE格式的网格文件来表示躯干的外观 -->
                 <mesh filename="${mesh_path}/trunk.dae" scale="1 1 1"/>
             </geometry>
         </visual>
+        <!-- 碰撞模型 (collision): 用于物理引擎中的碰撞检测 -->
         <collision>
             <origin rpy="0 0 0" xyz="0 0 0"/>
             <geometry>
+                <!-- 使用一个简单的长方体作为碰撞体 -->
                 <box size="${trunk_length} ${trunk_width} ${trunk_height}"/>
             </geometry>
         </collision>
+        <!-- 惯性参数 (inertial): 用于物理引擎中的动力学计算 -->
         <inertial>
             <origin rpy="0 0 0" xyz="${trunk_com_x} ${trunk_com_y} ${trunk_com_z}"/>
@@ -31,5 +50,15 @@
         </inertial>
     </link>
+    <!-- 实例化IMU宏，将其连接到 "base" 连杆上 -->
     <xacro:IMU connected_to="base" imu_name="base_imu" xyz="0. 0. 0." rpy="0. 0. 0."/>
+    <!-- 实例化四条腿 -->
+    <!--
+      `leg` 是在 leg.xacro 中定义的宏。
+      通过不同的参数（prefix, mirror, front_hind, origin）来生成四条不同位置和方向的腿。
+      - prefix: 关节和连杆名称的前缀 (e.g., "LF_HAA_joint")
+      - mirror: 镜像参数，用于翻转关节方向以创建左右腿
+      - front_hind: 前后参数，用于翻转关节方向以创建前后腿
+      - origin: 定义腿相对于基座原点的位置和姿态
+    -->
     <xacro:leg prefix="LF" mesh_path="${mesh_path}" mirror="1" mirror_dae="True" front_hind="1" front_hind_dae="True">
         <origin rpy="0 0 0" xyz="${leg_offset_x} ${leg_offset_y} 0"/>
