Commit message: add rviz display

File: legged_examples/legged_unitree/legged_unitree_description/urdf/common/leg.xacro (robot description, xacro)
@@ -33,5 +33,5 @@
                 </xacro:if>
                 <geometry>
-                    <mesh filename="${mesh_path}/hip.dae"
+                    <mesh filename="package://legged_unitree_description/meshes/$(arg robot_type)/hip.dae"
                           scale="1 1 1"/>
                 </geometry>
@@ -67,9 +67,9 @@
                 <geometry>
                     <xacro:if value="${mirror_dae == True}">
-                        <mesh filename="${mesh_path}/thigh.dae"
+                        <mesh filename="package://legged_unitree_description/meshes/$(arg robot_type)/thigh.dae"
                               scale="1 1 1"/>
                     </xacro:if>
                     <xacro:if value="${mirror_dae == False}">
-                        <mesh filename="${mesh_path}/thigh_mirror.dae"
+                        <mesh filename="package://legged_unitree_description/meshes/$(arg robot_type)/thigh_mirror.dae"
                               scale="1 1 1"/>
                     </xacro:if>
@@ -110,5 +110,5 @@
                 <origin rpy="0 0 0" xyz="0 0 0"/>
                 <geometry>
-                    <mesh filename="${mesh_path}/calf.dae"
+                     <mesh filename="package://legged_unitree_description/meshes/$(arg robot_type)/calf.dae"
                           scale="1 1 1"/>
                 </geometry>

Commit message: feat: 将四足机器人模型转换为轮腿式模型
此提交修改了机器人模型和控制系统，将四足机器人转换为轮腿式机器人。

主要变更包括：
- 修改了 URDF，用主动驱动的轮子替换了点状足端。
- 为轮式模型创建了一个新的 OCS2 任务配置，调整了状态/输入维度和成本函数。
- 实现了一个新的 `RollingConstraintCppAd` 来取代现有的零速约束，允许车轮滚动同时防止打滑。
- 更新了 C++ 控制器和接口代码，以处理具有16个驱动关节（12个腿部关节+4个车轮关节）的新机器人模型。

File: legged_examples/legged_unitree/legged_unitree_description/urdf/common/leg.xacro (robot description, xacro)
@@ -130,34 +130,36 @@
             </inertial>
         </link>
-        <joint name="${prefix}_foot_fixed" type="fixed" dont_collapse="true">
+        <joint name="${prefix}_WHEEL_JOINT" type="continuous">
             <origin rpy="0 0 0" xyz="0 0 ${-(calf_length)}"/>
             <parent link="${prefix}_calf"/>
-            <child link="${prefix}_FOOT"/>
+            <child link="${prefix}_WHEEL"/>
+            <axis xyz="0 1 0"/>
+            <dynamics damping="${damping}" friction="${friction}"/>
         </joint>
-        <link name="${prefix}_FOOT">
+        <link name="${prefix}_WHEEL">
+            <xacro:property name="wheel_radius" value="0.05"/>
+            <xacro:property name="wheel_width" value="0.02"/>
+            <xacro:property name="wheel_mass" value="0.1"/>
             <visual>
-                <origin rpy="0 0 0" xyz="0 0 0"/>
+                <origin rpy="${pi/2} 0 0" xyz="0 0 0"/>
                 <geometry>
-                    <sphere radius="${foot_radius-0.01}"/>
+                    <cylinder radius="${wheel_radius}" length="${wheel_width}"/>
                 </geometry>
                 <material name="orange"/>
             </visual>
             <collision>
-                <origin rpy="0 0 0" xyz="0 0 0"/>
+                <origin rpy="${pi/2} 0 0" xyz="0 0 0"/>
                 <geometry>
-                    <sphere radius="${foot_radius}"/>
+                    <cylinder radius="${wheel_radius}" length="${wheel_width}"/>
                 </geometry>
             </collision>
             <inertial>
-                <mass value="${foot_mass}"/>
-                <inertia
-                        ixx="${(2*foot_mass)/5.0*(foot_radius*foot_radius)}" ixy="0.0" ixz="0.0"
-                        iyy="${(2*foot_mass)/5.0*(foot_radius*foot_radius)}" iyz="0.0"
-                        izz="${(2*foot_mass)/5.0*(foot_radius*foot_radius)}"/>
+                <mass value="${wheel_mass}"/>
+                <xacro:property name="ixx" value="${(1/12) * wheel_mass * (3 * wheel_radius * wheel_radius + wheel_width * wheel_width)}"/>
+                <xacro:property name="iyy" value="${(1/2) * wheel_mass * wheel_radius * wheel_radius}"/>
+                <xacro:property name="izz" value="${(1/12) * wheel_mass * (3 * wheel_radius * wheel_radius + wheel_width * wheel_width)}"/>
+                <inertia ixx="${ixx}" ixy="0.0" ixz="0.0" iyy="${iyy}" iyz="0.0" izz="${izz}"/>
             </inertial>
         </link>
-        <gazebo reference="${prefix}_foot_fixed">
-            <disableFixedJointLumping>true</disableFixedJointLumping>
-        </gazebo>
         <gazebo reference="${prefix}_hip">
             <mu1>0.2</mu1>
@@ -178,7 +180,7 @@
             <self_collide>1</self_collide>
         </gazebo>
-        <gazebo reference="${prefix}_FOOT">
-            <mu1>0.6</mu1>
-            <mu2>0.6</mu2>
+        <gazebo reference="${prefix}_WHEEL">
+            <mu1>0.8</mu1>
+            <mu2>0.8</mu2>
             <self_collide>1</self_collide>
             <material>Gazebo/DarkGrey</material>

File: legged_examples/legged_unitree/legged_unitree_description/urdf/common/transmission.xacro (robot description, xacro)
@@ -32,4 +32,14 @@
             </actuator>
         </transmission>
+        <transmission name="${prefix}_WHEEL_JOINT_tran">
+            <type>transmission_interface/SimpleTransmission</type>
+            <joint name="${prefix}_WHEEL_JOINT">
+                <hardwareInterface>hardware_interface/EffortJointInterface</hardwareInterface>
+            </joint>
+            <actuator name="${prefix}_WHEEL_JOINT_motor">
+                <hardwareInterface>hardware_interface/EffortJointInterface</hardwareInterface>
+                <mechanicalReduction>1</mechanicalReduction>
+            </actuator>
+        </transmission>
     </xacro:macro>
 </robot>
